Commit message: fix empty collision warning on ROS noetic

File: urdf/hand_v0/hand.urdf.xacro (robot description, xacro)
@@ -231,4 +231,10 @@
                 <material name="body_sub" />
             </visual>
+            <collision>
+                <origin xyz="0.0 0.0 -0.01" rpy="0.0 0.0 0.0" />
+                <geometry>
+                    <box size="0.008 0.008 0.02"/>
+                </geometry>
+            </collision>
         </link>
     </xacro:macro>

File: urdf/sensors/pointgrey_chameleon.urdf.xacro (robot description, xacro)
@@ -15,4 +15,10 @@
                 </geometry>
             </visual>
+            <collision>
+                <origin xyz="0 0 0" rpy="0.0 0.0 0.0"/>
+                <geometry>
+                    <mesh filename="package://hsrb_meshes/meshes/sensors/head_camera.dae" />
+                </geometry>
+            </collision>
             <inertial>
                 <origin xyz="0 0 0"/>
